File: HW/ESP32_Eth_ADC_DAC/ESP32_Eth_ADC_DAC.kicad_pcb (KiCad board)
At the start: 2 copper layers, 4 parts, among them J1 2.54mm female 90deg, U1 ESP32-ETH01, U2 PCM5102A_dac, U3 WM8782S_adc

Commit message: Git fixed
Connections:
- U1 pad 19: /I2S_LRCLK -> /I2S_TX_LRCLK
- U1 pad 20: /I2S_bit_clock -> /I2S_TX_BCLK
- U1 pad 21: unconnected-(U1-IO36-Pad21) -> /I2S_RX_BCLK
- U1 pad 22: unconnected-(U1-IO39-Pad22) -> /I2S_RX_LRCLK
- U1 pad 24: /CLK_master -> unconnected-(U1-IO0-Pad24)
- U2 pad 1: unconnected-(U2-SCK-Pad1) -> GND
- U2 pad 2: /I2S_bit_clock -> /I2S_TX_BCLK
- U2 pad 4: /I2S_LRCLK -> /I2S_TX_LRCLK
- U2 pad 7: /I2S_LRCLK -> unconnected-(U2-LROUT-Pad7)
- U3 pad 1: /I2S_bit_clock -> /I2S_RX_BCLK
- U3 pad 2: /I2S_LRCLK -> /I2S_RX_LRCLK
- U3 pad 4: /CLK_master -> unconnected-(U3-CLK-Pad4)
Changed lines of the file:
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@@
 			(layers "*.Cu" "*.Mask")
 			(remove_unused_layers no)
-			(net "/I2S_LRCLK")
+			(net "/I2S_TX_LRCLK")
 			(pinfunction "IO14_19")
 			(pintype "bidirectional")
@@
 			(layers "*.Cu" "*.Mask")
 			(remove_unused_layers no)
-			(net "/I2S_bit_clock")
+			(net "/I2S_TX_BCLK")
 			(pinfunction "IO15_20")
 			(pintype "bidirectional")
@@
 			(layers "*.Cu" "*.Mask")
 			(remove_unused_layers no)
-			(net "unconnected-(U1-IO36-Pad21)")
+			(net "/I2S_RX_BCLK")
 			(pinfunction "IO36_21")
 			(pintype "input")
@@
 			(layers "*.Cu" "*.Mask")
 			(remove_unused_layers no)
-			(net "unconnected-(U1-IO39-Pad22)")
+			(net "/I2S_RX_LRCLK")
 			(pinfunction "IO39_22")
 			(pintype "input")
@@
 			(layers "*.Cu" "*.Mask")
 			(remove_unused_layers no)
-			(net "/CLK_master")
+			(net "unconnected-(U1-IO0-Pad24)")
 			(pinfunction "IO0_24")
 			(pintype "bidirectional")
@@
 			(layers "*.Cu" "*.Mask")
 			(remove_unused_layers no)
-			(net "/I2S_bit_clock")
+			(net "/I2S_RX_BCLK")
 			(pinfunction "B_1")
 			(pintype "output")
@@
 			(layers "*.Cu" "*.Mask")
 			(remove_unused_layers no)
-			(net "/I2S_LRCLK")
+			(net "/I2S_RX_LRCLK")
 			(pinfunction "LR_2")
 			(pintype "output")
@@
 			(layers "*.Cu" "*.Mask")
 			(remove_unused_layers no)
-			(net "/CLK_master")
+			(net "unconnected-(U3-CLK-Pad4)")
 			(pinfunction "CLK_4")
 			(pintype "output")
@@
 			(layers "*.Cu" "*.Mask")
 			(remove_unused_layers no)
-			(net "/CLK_master")
+			(net "unconnected-(U3-CLK-Pad4)")
 			(pinfunction "CLK_4")
 			(pintype "output")
@@
 			(layers "*.Cu" "*.Mask")
 			(remove_unused_layers no)
-			(net "/CLK_master")
+			(net "unconnected-(U3-CLK-Pad4)")
 			(pinfunction "CLK_4")
 			(pintype "output")
@@
 			(layers "*.Cu" "*.Mask")
 			(remove_unused_layers no)
-			(net "/CLK_master")
+			(net "unconnected-(U3-CLK-Pad4)")
 			(pinfunction "CLK_4")
 			(pintype "output")
@@
 			(layers "*.Cu" "*.Mask")
 			(remove_unused_layers no)
-			(net "unconnected-(U2-SCK-Pad1)")
+			(net "GND")
 			(pinfunction "SCK_1")
 			(pintype "input")
@@
 			(layers "*.Cu" "*.Mask")
 			(remove_unused_layers no)
-			(net "/I2S_bit_clock")
+			(net "/I2S_TX_BCLK")
 			(pinfunction "BCK_2")
 			(pintype "input")
@@
 			(layers "*.Cu" "*.Mask")
 			(remove_unused_layers no)
-			(net "/I2S_LRCLK")
+			(net "/I2S_TX_LRCLK")
 			(pinfunction "LCK_4")
 			(pintype "power_in")
@@
 			(layers "*.Cu" "*.Mask")
 			(remove_unused_layers no)
-			(net "/I2S_LRCLK")
+			(net "unconnected-(U2-LROUT-Pad7)")
 			(pinfunction "LROUT_7")
 			(pintype "power_in")
